Commit message: Preserve arm2 camera and grasp calibration

File: src/jetcobot_description/urdf/jetcobot.urdf (robot description, URDF)
Before this commit: robot jetcobot, 12 links, 11 joints
Joints:
- joint 3_Joint: limit lower=-2.3 upper=2.3 effort=0 velocity=0 -> lower=-2.8797932657906435 upper=2.8797932657906435 effort=0 velocity=0
- joint 4_Joint: limit lower=-2.6 upper=2.6 effort=0 velocity=0 -> lower=-2.8797932657906435 upper=2.8797932657906435 effort=0 velocity=0
- joint 5_Joint: limit lower=-2.5 upper=2.5 effort=0 velocity=0 -> lower=-2.8797932657906435 upper=2.8797932657906435 effort=0 velocity=0
- joint 6_Joint: limit lower=-2.84 upper=2.84 effort=0 velocity=0 -> lower=-3.0543261909900767 upper=3.0543261909900767 effort=0 velocity=0

Commit message: arm2 찐 최종

File: src/jetcobot_description/urdf/jetcobot.urdf (robot description, URDF)
Before this commit: robot jetcobot, 12 links, 11 joints
Joints:
- joint 1_Joint: limit lower=-3.14 upper=3.14 effort=0 velocity=0 -> lower=-2.9321531433504737 upper=2.9321531433504737 effort=0 velocity=0
- joint 2_Joint: limit lower=-2.9 upper=2.9 effort=0 velocity=0 -> lower=-2.443460952792061 upper=2.443460952792061 effort=0 velocity=0
- joint 3_Joint: limit lower=-2.3 upper=2.3 effort=0 velocity=0 -> lower=-2.6179938779914944 upper=2.6179938779914944 effort=0 velocity=0
- joint 4_Joint: limit lower=-2.6 upper=2.6 effort=0 velocity=0 -> lower=-2.6179938779914944 upper=2.6179938779914944 effort=0 velocity=0
- joint 5_Joint: limit lower=-2.5 upper=2.5 effort=0 velocity=0 -> lower=-2.705260340591211 upper=2.792526803190927 effort=0 velocity=0
- joint 6_Joint: limit lower=-2.84 upper=2.84 effort=0 velocity=0 -> lower=-3.141592653589793 upper=3.141592653589793 effort=0 velocity=0

Commit message: Update arm2 scan transfer and robot configuration

File: src/jetcobot_description/urdf/jetcobot.urdf (robot description, URDF)
Before this commit: robot jetcobot, 12 links, 11 joints
Joints:
- joint 6_Joint: limit lower=-3.141592653589793 upper=3.141592653589793 effort=0 velocity=0 -> lower=-2.6179938779914944 upper=2.6179938779914944 effort=0 velocity=0
